File: sch/sch.sch (KiCad schematic (older format))
At the start: 3 parts

Commit message: hoge
Parts:
- removed BT1: 30V, symbol Device:Battery_Cell
- removed R1: 5, symbol Device:R_US
- removed R2: 10, symbol Device:R_US
- added R? (x11): 30, symbol Device:R_US
- added R? (x6): 5, symbol Device:R_US
- added R? (x6): 15, symbol Device:R_US
- added R?: 10, symbol Device:R_US
- added R?: 20, symbol Device:R_US
Connections:
- wire segments 7 -> 70
